Commit message: Add navigation stack and tune robot simulation

File: robot_description/urdf/robot.urdf.xacro (robot description, xacro)
@@ -44,10 +44,4 @@
   <xacro:property name="wheel_y_bl"
                   value="${total_w/2.0 - wheel_len/2.0}"/>
-  <!-- ── Mid bogie wheels  (smaller passive rollers, between corners) -->
-  <xacro:property name="bogie_r"    value="0.03000"/>   <!-- [EST] 30 mm radius -->
-  <xacro:property name="bogie_len"  value="0.04500"/>   <!-- [EST] 45 mm axial  -->
-  <xacro:property name="bogie_mass" value="0.120"/>
-  <xacro:property name="bogie_z_bl" value="${bogie_r - chassis_cog_z}"/>
-  <xacro:property name="bogie_y_bl" value="${total_w/2.0 - bogie_len/2.0}"/>
   <!-- ── Top deck plate ──────────────────────────────────────────── -->
   <xacro:property name="deck_l"     value="0.22000"/>   <!-- [EST] -->
@@ -142,5 +136,5 @@
       <origin xyz="${x} ${y} ${z}" rpy="${pi/2} 0 0"/>
       <axis xyz="0 0 1"/>
-      <dynamics damping="0.05" friction="0.10"/>
+      <dynamics damping="0.10" friction="0.12"/>
     </joint>
   </xacro:macro>
@@ -194,15 +188,4 @@
                      x="${-wheel_x_bl}"  y="${-wheel_y_bl}" z="${wheel_z_bl}"/>
   <!-- ================================================================
-       7.  MID BOGIE WHEELS  (2 ×  passive continuous joints)
-       ================================================================ -->
-  <xacro:wheel_link name="mid_left_wheel"
-                    r="${bogie_r}" wlen="${bogie_len}" mass="${bogie_mass}"/>
-  <xacro:wheel_joint name="mid_left_wheel"  parent="base_link"
-                     x="0" y="${ bogie_y_bl}" z="${bogie_z_bl}"/>
-  <xacro:wheel_link name="mid_right_wheel"
-                    r="${bogie_r}" wlen="${bogie_len}" mass="${bogie_mass}"/>
-  <xacro:wheel_joint name="mid_right_wheel" parent="base_link"
-                     x="0" y="${-bogie_y_bl}" z="${bogie_z_bl}"/>
-  <!-- ================================================================
        8.  TOP DECK PLATE
        ================================================================ -->
@@ -479,6 +462,4 @@
   <xacro:wheel_gazebo name="rear_left_wheel"/>
   <xacro:wheel_gazebo name="rear_right_wheel"/>
-  <xacro:wheel_gazebo name="mid_left_wheel"/>
-  <xacro:wheel_gazebo name="mid_right_wheel"/>
   <!-- ── Skid-steer drive (front + rear driven pairs) ──────────────── -->
   <gazebo>
@@ -491,6 +472,6 @@
       <wheel_separation>${2.0 * wheel_y_bl}</wheel_separation>
       <wheel_radius>${wheel_r}</wheel_radius>
-      <topic>cmd_vel</topic>
-      <odom_topic>odom</odom_topic>
+      <topic>/cmd_vel</topic>
+      <odom_topic>/odom</odom_topic>
       <tf_topic>/tf</tf_topic>
       <frame_id>odom</frame_id>
@@ -503,5 +484,5 @@
     <plugin filename="gz-sim-joint-state-publisher-system"
             name="gz::sim::systems::JointStatePublisher">
-      <topic>joint_states</topic>
+      <topic>/joint_states</topic>
       <joint_name>pan_joint</joint_name>
       <joint_name>tilt_joint</joint_name>
@@ -510,6 +491,4 @@
       <joint_name>rear_left_wheel_joint</joint_name>
       <joint_name>rear_right_wheel_joint</joint_name>
-      <joint_name>mid_left_wheel_joint</joint_name>
-      <joint_name>mid_right_wheel_joint</joint_name>
     </plugin>
   </gazebo>
@@ -518,10 +497,10 @@
     <sensor name="lidar_sensor" type="gpu_lidar">
       <topic>scan</topic>
-      <update_rate>10</update_rate>
+      <update_rate>15</update_rate>
       <gz_frame_id>lidar_link</gz_frame_id>
       <lidar>
         <scan>
           <horizontal>
-            <samples>360</samples>
+            <samples>180</samples>
             <resolution>1</resolution>
             <min_angle>-3.14159265</min_angle>
@@ -531,5 +510,5 @@
         <range>
           <min>0.12</min>
-          <max>12.0</max>
+          <max>8.0</max>
           <resolution>0.01</resolution>
         </range>
@@ -541,5 +520,5 @@
       </lidar>
       <always_on>true</always_on>
-      <visualize>true</visualize>
+      <visualize>false</visualize>
     </sensor>
   </gazebo>

Commit message: navigation is working

File: robot_description/urdf/robot.urdf.xacro (robot description, xacro)
@@ -44,4 +44,6 @@
   <xacro:property name="wheel_y_bl"
                   value="${total_w/2.0 - wheel_len/2.0}"/>
+  <!-- Physical track width: 2 × wheel_y_bl = 2 × (0.23042/2 − 0.052/2) = 0.17842 m -->
+  <xacro:property name="drive_wheel_separation" value="0.17842"/>
   <!-- ── Top deck plate ──────────────────────────────────────────── -->
   <xacro:property name="deck_l"     value="0.22000"/>   <!-- [EST] -->
@@ -135,5 +137,5 @@
       <child  link="${name}"/>
       <origin xyz="${x} ${y} ${z}" rpy="${pi/2} 0 0"/>
-      <axis xyz="0 0 1"/>
+      <axis xyz="0 0 -1"/>
       <dynamics damping="0.10" friction="0.12"/>
     </joint>
@@ -268,4 +270,11 @@
     <origin xyz="-0.025 -0.040 ${deck_h/2.0 + lidar_h/2.0}" rpy="0 0 0"/>
   </joint>
+  <!-- Laser scan frame: ROS REP-103, X forward, Y left, Z up. -->
+  <link name="laser_link"/>
+  <joint name="laser_link_joint" type="fixed">
+    <parent link="lidar_link"/>
+    <child  link="laser_link"/>
+    <origin xyz="0 0 0" rpy="0 0 0"/>
+  </joint>
   <!-- ================================================================
        11.  ARM LOWER COLUMN  (fixed, 28.00 mm from side-view)
@@ -452,8 +461,9 @@
     <gazebo reference="${name}">
       <mu1>1.0</mu1>
-      <mu2>1.0</mu2>
-      <kp>1000000.0</kp>
-      <kd>100.0</kd>
-      <minDepth>0.001</minDepth>
+      <mu2>0.2</mu2>
+      <kp>200000.0</kp>
+      <kd>80.0</kd>
+      <minDepth>0.002</minDepth>
+      <maxVel>0.2</maxVel>
     </gazebo>
   </xacro:macro>
@@ -470,12 +480,13 @@
       <left_joint>rear_left_wheel_joint</left_joint>
       <right_joint>rear_right_wheel_joint</right_joint>
-      <wheel_separation>${2.0 * wheel_y_bl}</wheel_separation>
+      <wheel_separation>${drive_wheel_separation}</wheel_separation>
       <wheel_radius>${wheel_r}</wheel_radius>
       <topic>/cmd_vel</topic>
       <odom_topic>/odom</odom_topic>
-      <tf_topic>/tf</tf_topic>
+      <!-- EKF (robot_localization) owns odom→base_footprint TF; redirect gz TF so it does not conflict -->
+      <tf_topic>/gz/tf_unused</tf_topic>
       <frame_id>odom</frame_id>
       <child_frame_id>base_footprint</child_frame_id>
-      <odom_publish_frequency>30</odom_publish_frequency>
+      <odom_publish_frequency>50</odom_publish_frequency>
     </plugin>
   </gazebo>
@@ -485,4 +496,5 @@
             name="gz::sim::systems::JointStatePublisher">
       <topic>/joint_states</topic>
+      <update_rate>50</update_rate>
       <joint_name>pan_joint</joint_name>
       <joint_name>tilt_joint</joint_name>
@@ -494,13 +506,13 @@
   </gazebo>
   <!-- ── Deck LiDAR (2-D laser scan) ───────────────────────────────── -->
-  <gazebo reference="lidar_link">
+  <gazebo reference="laser_link">
     <sensor name="lidar_sensor" type="gpu_lidar">
       <topic>scan</topic>
-      <update_rate>15</update_rate>
-      <gz_frame_id>lidar_link</gz_frame_id>
+      <update_rate>20</update_rate>
+      <gz_frame_id>laser_link</gz_frame_id>
       <lidar>
         <scan>
           <horizontal>
-            <samples>180</samples>
+            <samples>360</samples>
             <resolution>1</resolution>
             <min_angle>-3.14159265</min_angle>
